Commit message: add camera
Signed-off-by: Kenji Brameld <kenjibrameld@gmail.com>

File: kaonashi_description/urdf/joints.xacro (robot description, xacro)
@@ -21,3 +21,13 @@
     <limit effort="1" lower="-3.1415" upper="3.1415" velocity="10.0"/>
   </joint>
+  <joint name="link3__camera" type="fixed">
+    <parent link="link3"/>
+    <child link="camera"/>
+    <origin rpy="0 0 0" xyz="0.0648 0 0"/>
+  </joint>
+  <joint name="camera__camera_optical" type="fixed">
+    <parent link="camera"/>
+    <child link="camera_optical"/>
+    <origin rpy="-1.57 0 -1.57" xyz="0 0 0"/>
+  </joint>
 </robot>

File: kaonashi_description/urdf/links.xacro (robot description, xacro)
@@ -42,4 +42,75 @@
     </visual>
   </link>
-  <link name="link3"/>
+  <link name="link3">
+    <visual>
+      <origin rpy="0 0 1.57" xyz="0.017 0 0"/>
+      <geometry>
+        <mesh filename="package://kaonashi_description/meshes/FPX330-S102.stl" scale="0.001 0.001 0.001"/>
+      </geometry>
+    </visual>
+    <visual>
+      <origin rpy="0 0 0" xyz="0.0205 0 0"/>
+      <geometry>
+        <box size="0.007 0.038 0.023"/>
+      </geometry>
+    </visual>
+    <visual>
+      <origin rpy="0 0 0" xyz="0.0275 0.0145 0"/>
+      <geometry>
+        <box size="0.007 0.009 0.038"/>
+      </geometry>
+    </visual>
+    <visual>
+      <origin rpy="0 0 0" xyz="0.0275 -0.0145 0"/>
+      <geometry>
+        <box size="0.007 0.009 0.038"/>
+      </geometry>
+    </visual>
+    <visual>
+      <origin rpy="0 1.57 0" xyz="0.037 0.014 0.014"/>
+      <geometry>
+        <cylinder radius="0.0025" length="0.012"/>
+      </geometry>
+    </visual>
+    <visual>
+      <origin rpy="0 1.57 0" xyz="0.037 -0.014 0.014"/>
+      <geometry>
+        <cylinder radius="0.0025" length="0.012"/>
+      </geometry>
+    </visual>
+    <visual>
+      <origin rpy="0 1.57 0" xyz="0.037 0.014 -0.014"/>
+      <geometry>
+        <cylinder radius="0.0025" length="0.012"/>
+      </geometry>
+    </visual>
+    <visual>
+      <origin rpy="0 1.57 0" xyz="0.037 -0.014 -0.014"/>
+      <geometry>
+        <cylinder radius="0.0025" length="0.012"/>
+      </geometry>
+    </visual>
+    <visual>
+      <origin rpy="0 0 0" xyz="0.0428 0 0"/>
+      <geometry>
+        <box size="0.0015 0.038 0.038"/>
+      </geometry>
+    </visual>
+    <visual>
+      <origin rpy="0 0 0" xyz="0.0452 0 0"/>
+      <geometry>
+        <box size="0.0032 0.020 0.020"/>
+      </geometry>
+    </visual>
+    <visual>
+      <origin rpy="0 1.57 0" xyz="0.0558 0 0"/>
+      <geometry>
+        <cylinder radius="0.007" length="0.018"/>
+      </geometry>
+    </visual>
+  </link>
+  <link name="camera">
+  </link>
+  <link name="camera_optical">
+  </link>
 </robot>
